Commit message: eod_robot_description/CMakeLists.txt

File: eod_robot_description/urdf/eod_robot_description.urdf (robot description, URDF)
Before this commit: robot eod_robot_description, 23 links, 22 joints
Links:
- added link world
Joints:
- added joint fixed_base_joint: type fixed, parent world, child base_link

Commit message: eod_robot_description

File: eod_robot_description/urdf/eod_robot_description.urdf (robot description, URDF)
Before this commit: robot eod_robot_description, 24 links, 23 joints
Joints:
- joint Arm_L1_joint: limit lower=-6.28 upper=6.28 effort=0 velocity=0 -> lower=-6.28 upper=6.28 effort=300 velocity=5
- joint Arm_L2_joint: limit lower=-6.28 upper=6.28 effort=0 velocity=0 -> lower=-6.28 upper=6.28 effort=300 velocity=5
- joint Arm_L3_joint: limit lower=-6.28 upper=6.28 effort=0 velocity=0 -> lower=-6.28 upper=6.28 effort=300 velocity=5
- joint Arm_L4_joint: limit lower=-6.28 upper=6.28 effort=0 velocity=0 -> lower=-6.28 upper=6.28 effort=100 velocity=5
- joint Arm_L5_joint: limit lower=-6.28 upper=6.28 effort=0 velocity=0 -> lower=-6.28 upper=6.28 effort=100 velocity=5
- joint Arm_L6_joint: limit lower=-6.28 upper=6.28 effort=0 velocity=0 -> lower=-6.28 upper=6.28 effort=100 velocity=5
- joint Arm_R1_joint: limit lower=-6.28 upper=6.28 effort=0 velocity=0 -> lower=-6.28 upper=6.28 effort=300 velocity=5
- joint Arm_R2_joint: limit lower=-6.28 upper=6.28 effort=0 velocity=0 -> lower=-6.28 upper=6.28 effort=300 velocity=5
- joint Arm_R3_joint: limit lower=-6.28 upper=6.28 effort=0 velocity=0 -> lower=-6.28 upper=6.28 effort=300 velocity=5
- joint Arm_R4_joint: limit lower=-6.28 upper=6.28 effort=0 velocity=0 -> lower=-6.28 upper=6.28 effort=100 velocity=5
- joint Arm_R5_joint: limit lower=-6.28 upper=6.28 effort=0 velocity=0 -> lower=-6.28 upper=6.28 effort=100 velocity=5
- joint Arm_R6_joint: limit lower=-6.28 upper=6.28 effort=0 velocity=0 -> lower=-6.28 upper=6.28 effort=100 velocity=5

Commit message: gazebo

File: eod_robot_description/urdf/eod_robot_description.urdf (robot description, URDF)
Before this commit: robot eod_robot_description, 24 links, 23 joints
Joints:
- joint Arm_L6_joint: limit lower=-6.28 upper=6.28 effort=100 velocity=5 -> effort=100 velocity=5; type revolute -> continuous
- joint Arm_R6_joint: limit lower=-6.28 upper=6.28 effort=100 velocity=5 -> effort=100 velocity=5; type revolute -> continuous
- joint gripper_finger1_finger_tip_joint: mimic joint=gripper_finger1_joint multiplier=1.49462955 -> joint=gripper_finger1_joint multiplier=1.49462955 offset=0
- joint gripper_finger2_finger_tip_joint: mimic joint=gripper_finger1_joint multiplier=1.49462955 -> joint=gripper_finger1_joint multiplier=1.49462955 offset=0
- joint gripper_finger2_joint: mimic joint=gripper_finger1_joint -> joint=gripper_finger1_joint multiplier=0.4563942 offset=0

Commit message: urdf

File: eod_robot_description/urdf/eod_robot_description.urdf (robot description, URDF)
Before this commit: robot eod_robot_description, 24 links, 23 joints
Links:
- added link camera_color_frame
- added link camera_color_optical_frame
- added link camera_depth_frame
- added link camera_depth_optical_frame
- added link camera_left_ir_frame
- added link camera_left_ir_optical_frame
- added link camera_link, mass 0.564; collision box size=0.02505 0.09 0.025; visual mesh filename=package://eod_robot_description/meshes/d435.dae
- added link camera_right_ir_frame
- added link camera_right_ir_optical_frame
- added link right_camera_color_frame
- added link right_camera_color_optical_frame
- added link right_camera_depth_frame
- added link right_camera_depth_optical_frame
- added link right_camera_left_ir_frame
- added link right_camera_left_ir_optical_frame
- added link right_camera_link, mass 0.564; collision box size=0.02505 0.09 0.025; visual mesh filename=package://eod_robot_description/meshes/d435.dae
- added link right_camera_right_ir_frame
- added link right_camera_right_ir_optical_frame
Joints:
- added joint base_camera_joint: type fixed, parent base_link, child camera_link, origin xyz=0.09884 -0.0175 0.03381 rpy=3.14159 0.00 0.00 
- added joint camera_color_joint: type fixed, parent camera_depth_frame, child camera_color_frame, origin xyz=0 0.015 0 rpy=0 0 0
- added joint camera_color_optical_joint: type fixed, parent camera_color_frame, child camera_color_optical_frame, origin xyz=0 0 0 rpy=-1.57079632679 0 -1.57079632679
- added joint camera_depth_joint: type fixed, parent camera_link, child camera_depth_frame, origin xyz=0 0 0 rpy=0 0 0
- added joint camera_depth_optical_joint: type fixed, parent camera_depth_frame, child camera_depth_optical_frame, origin xyz=0 0 0 rpy=-1.57079632679 0 -1.57079632679
- added joint camera_left_ir_joint: type fixed, parent camera_depth_frame, child camera_left_ir_frame, origin xyz=0 0.0 0 rpy=0 0 0
- added joint camera_left_ir_optical_joint: type fixed, parent camera_left_ir_frame, child camera_left_ir_optical_frame, origin xyz=0 0 0 rpy=-1.57079632679 0 -1.57079632679
- added joint camera_right_ir_joint: type fixed, parent camera_depth_frame, child camera_right_ir_frame, origin xyz=0 -0.05 0 rpy=0 0 0
- added joint camera_right_ir_optical_joint: type fixed, parent camera_right_ir_frame, child camera_right_ir_optical_frame, origin xyz=0 0 0 rpy=-1.57079632679 0 -1.57079632679
- added joint right_base_camera_joint: type fixed, parent Arm_R6_link, child right_camera_link, origin xyz=-0.027 0.0812 -0.0515 rpy=0.18 0.00 1.57079632679 
- added joint right_camera_color_joint: type fixed, parent right_camera_depth_frame, child right_camera_color_frame, origin xyz=0 0.015 0 rpy=0 0 0
- added joint right_camera_color_optical_joint: type fixed, parent right_camera_color_frame, child right_camera_color_optical_frame, origin xyz=0 0 0 rpy=-1.57079632679 0 -1.57079632679
- added joint right_camera_depth_joint: type fixed, parent right_camera_link, child right_camera_depth_frame, origin xyz=0 0 0 rpy=0 0 0
- added joint right_camera_depth_optical_joint: type fixed, parent right_camera_depth_frame, child right_camera_depth_optical_frame, origin xyz=0 0 0 rpy=-1.57079632679 0 -1.57079632679
- added joint right_camera_left_ir_joint: type fixed, parent right_camera_depth_frame, child right_camera_left_ir_frame, origin xyz=0 0.0 0 rpy=0 0 0
- added joint right_camera_left_ir_optical_joint: type fixed, parent right_camera_left_ir_frame, child right_camera_left_ir_optical_frame, origin xyz=0 0 0 rpy=-1.57079632679 0 -1.57079632679
- added joint right_camera_right_ir_joint: type fixed, parent right_camera_depth_frame, child right_camera_right_ir_frame, origin xyz=0 -0.05 0 rpy=0 0 0
- added joint right_camera_right_ir_optical_joint: type fixed, parent right_camera_right_ir_frame, child right_camera_right_ir_optical_frame, origin xyz=0 0 0 rpy=-1.57079632679 0 -1.57079632679

Commit message: urdf

File: eod_robot_description/urdf/eod_robot_description.urdf (robot description, URDF)
Before this commit: robot eod_robot_description, 42 links, 41 joints
Links:
- added link left_camera_color_frame
- added link left_camera_color_optical_frame
- added link left_camera_depth_frame
- added link left_camera_depth_optical_frame
- added link left_camera_left_ir_frame
- added link left_camera_left_ir_optical_frame
- added link left_camera_link, mass 0.564; collision box size=0.02505 0.09 0.025; visual mesh filename=package://eod_robot_description/meshes/d435.dae
- added link left_camera_right_ir_frame
- added link left_camera_right_ir_optical_frame
Joints:
- added joint left_base_camera_joint: type fixed, parent Arm_L6_link_add, child left_camera_link, origin xyz=-0.027 0.0815 -0.0515 rpy=0.18 0.00 1.57079632679
- added joint left_camera_color_joint: type fixed, parent left_camera_depth_frame, child left_camera_color_frame, origin xyz=0 0.015 0 rpy=0 0 0
- added joint left_camera_color_optical_joint: type fixed, parent left_camera_color_frame, child left_camera_color_optical_frame, origin xyz=0 0 0 rpy=-1.57079632679 0 -1.57079632679
- added joint left_camera_depth_joint: type fixed, parent left_camera_link, child left_camera_depth_frame, origin xyz=0 0 0 rpy=0 0 0
- added joint left_camera_depth_optical_joint: type fixed, parent left_camera_depth_frame, child left_camera_depth_optical_frame, origin xyz=0 0 0 rpy=-1.57079632679 0 -1.57079632679
- added joint left_camera_left_ir_joint: type fixed, parent left_camera_depth_frame, child left_camera_left_ir_frame, origin xyz=0 0.0 0 rpy=0 0 0
- added joint left_camera_left_ir_optical_joint: type fixed, parent left_camera_left_ir_frame, child left_camera_left_ir_optical_frame, origin xyz=0 0 0 rpy=-1.57079632679 0 -1.57079632679
- added joint left_camera_right_ir_joint: type fixed, parent left_camera_depth_frame, child left_camera_right_ir_frame, origin xyz=0 -0.05 0 rpy=0 0 0
- added joint left_camera_right_ir_optical_joint: type fixed, parent left_camera_right_ir_frame, child left_camera_right_ir_optical_frame, origin xyz=0 0 0 rpy=-1.57079632679 0 -1.57079632679
- joint base_camera_joint: origin xyz=0.09884 -0.0175 0.03381 rpy=3.14159 0.00 0.00  -> xyz=0.1 -0.0175 0.03381 rpy=3.14159 0.00 0.00 
- joint right_base_camera_joint: origin xyz=-0.027 0.0812 -0.0515 rpy=0.18 0.00 1.57079632679  -> xyz=-0.027 0.0815 -0.0515 rpy=0.18 0.00 1.57079632679 

Commit message: vehicle

File: eod_robot_description/urdf/eod_robot_description.urdf (robot description, URDF)
Before this commit: robot eod_robot_description, 51 links, 50 joints
Links:
- added link left_back_wheel; visual cylinder length=0.06 radius=0.098
- added link left_front_wheel; visual cylinder length=0.06 radius=0.098
- added link right_back_wheel; visual cylinder length=0.06 radius=0.098
- added link right_front_wheel; visual cylinder length=0.06 radius=0.098
Joints:
- added joint left_back_wheel_joint: type continuous, parent base_link, child left_back_wheel, origin xyz=-0.602 0.2765 -0.402 rpy=0 0 0, axis 0 1 0, limit effort=100 velocity=100
- added joint left_front_wheel_joint: type continuous, parent base_link, child left_front_wheel, origin xyz=-0.062 0.2765 -0.402 rpy=0 0 0, axis 0 1 0, limit effort=100 velocity=100
- added joint right_back_wheel_joint: type continuous, parent base_link, child right_back_wheel, origin xyz=-0.602 -0.276 -0.402 rpy=0 0 0, axis 0 1 0, limit effort=100 velocity=100
- added joint right_front_wheel_joint: type continuous, parent base_link, child right_front_wheel, origin xyz=-0.062 -0.2765 -0.402 rpy=0 0 0, axis 0 1 0, limit effort=100 velocity=100

Commit message: urdf

File: eod_robot_description/urdf/eod_robot_description.urdf (robot description, URDF)
Before this commit: robot eod_robot_description, 55 links, 54 joints
Links:
- link left_back_wheel: mass None -> 2; geometry collision cylinder length=0.06 radius=0.098; visual cylinder length=0.06 radius=0.098
- link left_front_wheel: mass None -> 2; geometry collision cylinder length=0.06 radius=0.098; visual cylinder length=0.06 radius=0.098
- link right_back_wheel: mass None -> 2; geometry collision cylinder length=0.06 radius=0.098; visual cylinder length=0.06 radius=0.098
- link right_front_wheel: mass None -> 2; geometry collision cylinder length=0.06 radius=0.098; visual cylinder length=0.06 radius=0.098

Commit message: vehicle

File: eod_robot_description/urdf/eod_robot_description.urdf (robot description, URDF)
Before this commit: robot eod_robot_description, 55 links, 54 joints
Links:
- removed link world
Joints:
- removed joint fixed_base_joint
