Commit message: camera

File: eod_robot_description/urdf/eod_robot_description_cameras.xacro (robot description, xacro)
@@ -3,23 +3,15 @@
 <xacro:macro name="cameras">
 <!--vehicle_camera-->
-  <link name="camera_link">
+  <link name="vehicle_camera_link">
     <visual>
-      <origin
-        rpy="1.57079632679 0 1.57079632679"
-        xyz="0.0149 -0.0175 0"/>
-      <geometry>
-        <!-- <box size="${d435_cam_width} ${d435_cam_height} ${d435_cam_depth}"/> -->
-        <mesh
-          filename="package://eod_robot_description/meshes/d435.dae"/>
-        <!--<mesh filename="package://realsense2_description/meshes/d435/d435.dae" />-->
-      </geometry>
-      <material name="">
-        <color rgba="1 0 0 1" />
+      <origin rpy="1.57079632679 0.00 1.57079632679" xyz="0.0149 0.0175 0"/>
+      <geometry>
+        <mesh filename="package://eod_robot_description/meshes/d435.dae"/>
+      </geometry>
+        <material name=""> <color rgba="1 0 0 1" />
       </material>
     </visual>
     <collision>
-      <origin
-        rpy="0 0 0"
-        xyz="0 -0.0175 0"/>
+      <origin rpy="0 0 0" xyz="0 0.0175 0"/>
       <geometry>
         <box size="0.02505 0.09 0.025"/>
@@ -27,93 +19,46 @@
     </collision>
     <inertial>
-      <!-- The following are not reliable values, and should not be used for modeling -->
       <mass value="0.564"/>
       <origin xyz="0 0 0"/>
-      <inertia
-        ixx="0.003881243"
-        ixy="0.0"
-        ixz="0.0"
-        iyy="0.000498940"
-        iyz="0.0"
-        izz="0.003879257"/>
+      <inertia ixx="0.003881243"  ixy="0.0" ixz="0.0" iyy="0.000498940" iyz="0.0" izz="0.003879257"/>
     </inertial>
   </link>
   <joint name="base_camera_joint" type="fixed">
+    <origin xyz="0.1 -0.0175 0.03381" rpy="0.00 0.00 0.00 "/>
+    <parent link="base_link"/>
+    <child link="vehicle_camera_link"/>
+  </joint >
+  <joint name="vehicle_camera_depth_joint" type="fixed">
+    <origin rpy="0 0 0" xyz="0 0 0"/>
+    <parent link="vehicle_camera_link"/>
+    <child link="vehicle_camera_depth_frame"/>
+  </joint>
+  <link name="vehicle_camera_depth_frame">
+    <inertial>
+      <mass value="0.001" />
+      <origin rpy="0 0 0" xyz="0 0 0" />
+      <inertia ixx="0.0001" ixy="0.0" ixz="0.0"
+              iyy="0.0001" iyz="0.0"
+              izz="0.0001" />
+    </inertial>
+  </link>
+  <joint name="vehicle_camera_depth_optical_joint" type="fixed">
     <origin
-      xyz="0.1 -0.0175 0.03381"
-      rpy="3.14159 0.00 0.00 "/>
-    <parent link="base_link"/>
-    <child link="camera_link"/>
-  </joint >
-  <joint name="camera_depth_joint" type="fixed">
-    <origin
-      rpy="0 0 0"
-      xyz="0 0 0"/>
-    <parent link="camera_link"/>
-    <child link="camera_depth_frame"/>
-  </joint>
-  <link name="camera_depth_frame"/>
-  <joint name="camera_depth_optical_joint" type="fixed">
-    <origin
-      rpy="-1.57079632679 0 -1.57079632679"
-      xyz="0 0 0"/>
-    <parent link="camera_depth_frame"/>
-    <child link="camera_depth_optical_frame"/>
-  </joint>
-  <link name="camera_depth_optical_frame"/>
-<!-- camera left IR joints and links -->
-  <joint name="camera_left_ir_joint" type="fixed">
-    <origin
-      rpy="0 0 0"
-      xyz="0 0.0 0"/>
-    <parent link="camera_depth_frame"/>
-    <child link="camera_left_ir_frame"/>
-  </joint>
-  <link name="camera_left_ir_frame"/>
-  <joint name="camera_left_ir_optical_joint" type="fixed">
-    <origin
-      rpy="-1.57079632679 0 -1.57079632679"
-      xyz="0 0 0"/>
-    <parent link="camera_left_ir_frame"/>
-    <child link="camera_left_ir_optical_frame"/>
-  </joint>
-  <link name="camera_left_ir_optical_frame"/>
-  <!-- camera right IR joints and links -->
-  <joint name="camera_right_ir_joint" type="fixed">
-    <origin
-      rpy="0 0 0"
-      xyz="0 -0.05 0"/>
-    <parent link="camera_depth_frame"/>
-    <child link="camera_right_ir_frame"/>
-  </joint>
-  <link name="camera_right_ir_frame"/>
-  <joint name="camera_right_ir_optical_joint" type="fixed">
-    <origin
-      rpy="-1.57079632679 0 -1.57079632679"
-      xyz="0 0 0"/>
-    <parent link="camera_right_ir_frame"/>
-    <child link="camera_right_ir_optical_frame"/>
-  </joint>
-  <link name="camera_right_ir_optical_frame"/>
-  <!-- camera color joints and links -->
-  <joint name="camera_color_joint" type="fixed">
-    <origin
-      rpy="0 0 0"
-      xyz="0 0.015 0"/>
-    <parent link="camera_depth_frame"/>
-    <child link="camera_color_frame"/>
-  </joint>
-  <link name="camera_color_frame"/>
-  <joint name="camera_color_optical_joint" type="fixed">
-   <origin
-     rpy="-1.57079632679 0 -1.57079632679"
-     xyz="0 0 0"/>
-   <parent link="camera_color_frame"/>
-   <child link="camera_color_optical_frame"/>
- </joint>
-  <link name="camera_color_optical_frame"/>
+      rpy="-1.57079632679 0 -1.57079632679" xyz="0 0 0"/>
+    <parent link="vehicle_camera_depth_frame"/>
+    <child link="vehicle_camera_depth_optical_frame"/>
+  </joint>
+  <link name="vehicle_camera_depth_optical_frame">
+    <inertial>
+      <mass value="0.001" />
+      <origin rpy="0 0 0"  xyz="0 0 0" />
+      <inertia ixx="0.0001" ixy="0.0" ixz="0.0"
+              iyy="0.0001" iyz="0.0"
+              izz="0.0001" />
+    </inertial>
+  </link>
 <!--right_camera-->
 <joint name="right_base_camera_joint" type="fixed">
-	  <origin xyz="-0.027 0.0815 -0.0515" rpy="0.18 0.00 1.57079632679 "/>
+    <origin xyz="-0.027 0.0815 -0.0515" rpy="-2.9615926 0.00 1.57079632679 "/>
     <parent link="Arm_R6_link"/>
 	  <child link="right_camera_link"/>
@@ -121,17 +66,14 @@
   <link name="right_camera_link">
     <visual>
-      <origin rpy="1.57079632679 0 1.57079632679" xyz="0.0149 -0.0175 0"/>
-      <geometry>
-        <!-- <box size="${d435_cam_width} ${d435_cam_height} ${d435_cam_depth}"/> -->
+       <origin rpy="1.57079632679 0.00 1.57079632679" xyz="0.0149 0.0175 0"/>
+      <geometry>
         <mesh filename="package://eod_robot_description/meshes/d435.dae"/>
-        <!--<mesh filename="package://realsense2_description/meshes/d435/d435.dae" />-->
-      </geometry>
-            <material
-        name="">
-        <color rgba="1 0 0 1" />
+      </geometry>
+      <material
+        name=""> <color rgba="1 0 0 1" />
       </material>
     </visual>
     <collision>
-      <origin rpy="0 0 0" xyz="0 -0.0175 0"/>
+      <origin rpy="0 0 0" xyz="0 0.0175 0"/>
       <geometry>
         <box size="0.02505 0.09 0.025"/>
@@ -139,5 +81,4 @@
     </collision>
     <inertial>
-      <!-- The following are not reliable values, and should not be used for modeling -->
       <mass value="0.564"/>
       <origin xyz="0 0 0"/>
@@ -145,5 +86,4 @@
     </inertial>
   </link>
-  <!-- camera depth joints and links -->
   <joint name="right_camera_depth_joint" type="fixed">
     <origin rpy="0 0 0" xyz="0 0 0"/>
@@ -151,5 +91,13 @@
     <child link="right_camera_depth_frame"/>
   </joint>
-  <link name="right_camera_depth_frame"/>
+  <link name="right_camera_depth_frame">
+    <inertial>
+      <mass value="0.001" />
+      <origin xyz="0 0 0" />
+      <inertia ixx="0.0001" ixy="0.0" ixz="0.0"
+              iyy="0.0001" iyz="0.0"
+              izz="0.0001" />
+    </inertial>
+  </link>
   <joint name="right_camera_depth_optical_joint" type="fixed">
     <origin rpy="-1.57079632679 0 -1.57079632679" xyz="0 0 0"/>
@@ -157,47 +105,16 @@
     <child link="right_camera_depth_optical_frame"/>
   </joint>
-  <link name="right_camera_depth_optical_frame"/>
-  <!-- camera left IR joints and links -->
-  <joint name="right_camera_left_ir_joint" type="fixed">
-    <origin rpy="0 0 0" xyz="0 0.0 0"/>
-    <parent link="right_camera_depth_frame"/>
-    <child link="right_camera_left_ir_frame"/>
-  </joint>
-  <link name="right_camera_left_ir_frame"/>
-  <joint name="right_camera_left_ir_optical_joint" type="fixed">
-    <origin rpy="-1.57079632679 0 -1.57079632679" xyz="0 0 0"/>
-    <parent link="right_camera_left_ir_frame"/>
-    <child link="right_camera_left_ir_optical_frame"/>
-  </joint>
-  <link name="right_camera_left_ir_optical_frame"/>
-  <!-- camera right IR joints and links -->
-  <joint name="right_camera_right_ir_joint" type="fixed">
-    <origin rpy="0 0 0" xyz="0 -0.05 0"/>
-    <parent link="right_camera_depth_frame"/>
-    <child link="right_camera_right_ir_frame"/>
-  </joint>
-  <link name="right_camera_right_ir_frame"/>
-  <joint name="right_camera_right_ir_optical_joint" type="fixed">
-    <origin rpy="-1.57079632679 0 -1.57079632679" xyz="0 0 0"/>
-    <parent link="right_camera_right_ir_frame"/>
-    <child link="right_camera_right_ir_optical_frame"/>
-  </joint>
-  <link name="right_camera_right_ir_optical_frame"/>
-  <!-- camera color joints and links -->
-  <joint name="right_camera_color_joint" type="fixed">
-    <origin rpy="0 0 0" xyz="0 0.015 0"/>
-    <parent link="right_camera_depth_frame"/>
-    <child link="right_camera_color_frame"/>
-  </joint>
-  <link name="right_camera_color_frame"/>
-  <joint name="right_camera_color_optical_joint" type="fixed">
-    <origin rpy="-1.57079632679 0 -1.57079632679" xyz="0 0 0"/>
-    <parent link="right_camera_color_frame"/>
-    <child link="right_camera_color_optical_frame"/>
-  </joint>
-  <link name="right_camera_color_optical_frame"/>
+  <link name="right_camera_depth_optical_frame">
+    <inertial>
+      <mass value="0.001" />
+      <origin xyz="0 0 0" />
+      <inertia ixx="0.0001" ixy="0.0" ixz="0.0"
+              iyy="0.0001" iyz="0.0"
+              izz="0.0001" />
+    </inertial>
+  </link>
 <!--left_camera-->
 <joint name="left_base_camera_joint" type="fixed">
-	<origin xyz="-0.027 0.0815 -0.0515" rpy="0.18 0.00 1.57079632679"/>
+	<origin xyz="-0.027 0.0815 -0.0515" rpy="-2.9615926 0.00 1.57079632679"/>
 	<parent link="Arm_L6_link_add"/>
 	<child link="left_camera_link"/>
@@ -205,14 +122,12 @@
   <link name="left_camera_link">
     <visual>
-      <origin rpy="1.57079632679 0 1.57079632679" xyz="0.0149 -0.0175 0"/>
-      <geometry>
-        <!-- <box size="${d435_cam_width} ${d435_cam_height} ${d435_cam_depth}"/> -->
+      <origin rpy="1.57079632679 0.00 1.57079632679" xyz="0.0149 0.0175 0"/>
+      <geometry>
         <mesh filename="package://eod_robot_description/meshes/d435.dae"/>
-        <!--<mesh filename="package://realsense2_description/meshes/d435/d435.dae" />-->
       </geometry>
       <material name="camera_aluminum"/>
     </visual>
     <collision>
-      <origin rpy="0 0 0" xyz="0 -0.0175 0"/>
+      <origin rpy="0 0 0" xyz="0 0.0175 0"/>
       <geometry>
         <box size="0.02505 0.09 0.025"/>
@@ -220,5 +135,4 @@
     </collision>
     <inertial>
-      <!-- The following are not reliable values, and should not be used for modeling -->
       <mass value="0.564"/>
       <origin xyz="0 0 0"/>
@@ -232,5 +146,13 @@
     <child link="left_camera_depth_frame"/>
   </joint>
-  <link name="left_camera_depth_frame"/>
+  <link name="left_camera_depth_frame">
+    <inertial>
+      <mass value="0.001" />
+      <origin xyz="0 0 0" />
+      <inertia ixx="0.0001" ixy="0.0" ixz="0.0"
+              iyy="0.0001" iyz="0.0"
+              izz="0.0001" />
+    </inertial>
+  </link>
   <joint name="left_camera_depth_optical_joint" type="fixed">
     <origin rpy="-1.57079632679 0 -1.57079632679" xyz="0 0 0"/>
@@ -238,45 +160,14 @@
     <child link="left_camera_depth_optical_frame"/>
   </joint>
-  <link name="left_camera_depth_optical_frame"/>
-  <!-- camera left IR joints and links -->
-  <joint name="left_camera_left_ir_joint" type="fixed">
-    <origin rpy="0 0 0" xyz="0 0.0 0"/>
-    <parent link="left_camera_depth_frame"/>
-    <child link="left_camera_left_ir_frame"/>
-  </joint>
-  <link name="left_camera_left_ir_frame"/>
-  <joint name="left_camera_left_ir_optical_joint" type="fixed">
-    <origin rpy="-1.57079632679 0 -1.57079632679" xyz="0 0 0"/>
-    <parent link="left_camera_left_ir_frame"/>
-    <child link="left_camera_left_ir_optical_frame"/>
-  </joint>
-  <link name="left_camera_left_ir_optical_frame"/>
-  <!-- camera right IR joints and links -->
-  <joint name="left_camera_right_ir_joint" type="fixed">
-    <origin rpy="0 0 0" xyz="0 -0.05 0"/>
-    <parent link="left_camera_depth_frame"/>
-    <child link="left_camera_right_ir_frame"/>
-  </joint>
-  <link name="left_camera_right_ir_frame"/>
-  <joint name="left_camera_right_ir_optical_joint" type="fixed">
-    <origin rpy="-1.57079632679 0 -1.57079632679" xyz="0 0 0"/>
-    <parent link="left_camera_right_ir_frame"/>
-    <child link="left_camera_right_ir_optical_frame"/>
-  </joint>
-  <link name="left_camera_right_ir_optical_frame"/>
-  <!-- camera color joints and links -->
-  <joint name="left_camera_color_joint" type="fixed">
-      <origin rpy="0 0 0" xyz="0 0.015 0"/>
-      <parent link="left_camera_depth_frame"/>
-      <child link="left_camera_color_frame"/>
-  </joint>
-  <link name="left_camera_color_frame"/>
-<joint name="left_camera_color_optical_joint" type="fixed">
-    <origin rpy="-1.57079632679 0 -1.57079632679" xyz="0 0 0"/>
-    <parent link="left_camera_color_frame"/>
-    <child link="left_camera_color_optical_frame"/>
-  </joint>
-  <link name="left_camera_color_optical_frame"/>
-  <gazebo reference="camera_link">
+  <link name="left_camera_depth_optical_frame">
+    <inertial>
+      <mass value="0.001" />
+      <origin xyz="0 0 0" />
+      <inertia ixx="0.0001" ixy="0.0" ixz="0.0"
+              iyy="0.0001" iyz="0.0"
+              izz="0.0001" />
+    </inertial>
+  </link>
+  <gazebo reference="vehicle_camera_link">
     <implicitSpringDamper>1</implicitSpringDamper>
     <mu1>100000</mu1>
@@ -284,5 +175,5 @@
     <kp>100000000.0</kp>
     <kd>1.0</kd>
-    <material>Gazebo/Green</material>
+    <material>Gazebo/GreenTransparent</material>
   </gazebo>
   <gazebo reference="right_camera_link">
@@ -292,5 +183,5 @@
     <kp>100000000.0</kp>
     <kd>1.0</kd>
-    <material>Gazebo/Red</material>
+    <material>Gazebo/RedTransparent</material>
   </gazebo>
   <gazebo reference="left_camera_link">
@@ -300,6 +191,129 @@
     <kp>100000000.0</kp>
     <kd>1.0</kd>
-    <material>Gazebo/Red</material>
+    <material>Gazebo/RedTransparent</material>
   </gazebo>
+<gazebo reference="vehicle_camera_link">
+  <sensor name="vehicle_camera_link_camera" type="depth">
+    <update_rate>20</update_rate>
+    <camera>
+      <horizontal_fov>1.047198</horizontal_fov>
+      <image>
+        <width>640</width>
+        <height>480</height>
+        <format>R8G8B8</format>
+      </image>
+      <clip>
+        <near>0.05</near>
+        <far>8.0</far>
+      </clip>
+    </camera>
+    <plugin name="vehicle_camera_controller" filename="libgazebo_ros_openni_kinect.so">
+      <robotNamespace>/eod_robot_description</robotNamespace>
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