Commit message: temp

File: eod_robot_description/urdf/eod_robot_description_left_arm.xacro (robot description, xacro)
@@ -215,5 +215,5 @@
     type="fixed">
     <origin xyz="0 0 0" rpy="0 -2.1991 0" />
-    <parent link="Arm_L6_link" />
+    <parent link="6=[" />
     <child link="Arm_L6_link_add" />
     <axis xyz="0 1 0" />

Commit message: effector

File: eod_robot_description/urdf/eod_robot_description_left_arm.xacro (robot description, xacro)
@@ -211,11 +211,15 @@
     </collision>
   </link>
- <joint
-    name="Arm_L6_joint_add"
-    type="fixed">
+ <joint name="Arm_L6_joint_add" type="fixed">
     <origin xyz="0 0 0" rpy="0 -2.1991 0" />
-    <parent link="6=[" />
+    <parent link="Arm_L6_link" />
     <child link="Arm_L6_link_add" />
     <axis xyz="0 1 0" />
+  </joint>
+<link name="Arm_L_end_effector" />
+ <joint name="Arm_L_end_effector_joint" type="fixed">
+    <origin xyz="0.001 0.17232 -0.00343" rpy="1.5360 0.4083 3.1307" />
+    <parent link="Arm_L6_link" />
+    <child link="Arm_L_end_effector" />
   </joint>
   <transmission name="Arm_L1_trans">

File: eod_robot_description/urdf/eod_robot_description_right_arm.xacro (robot description, xacro)
@@ -189,4 +189,10 @@
     <limit effort="100" velocity="5" />
   </joint>
+  <link name="Arm_R_end_effector" />
+  <joint name="Arm_R_end_effector_joint" type="fixed">
+    <origin xyz="0 0.26797 0" rpy="-1.5708 -1.4008 0" />
+    <parent link="Arm_R6_link" />
+    <child link="Arm_R_end_effector" />
+   </joint>
   <transmission name="Arm_R1_trans">
     <type>transmission_interface/SimpleTransmission</type>

Commit message: effecor

File: eod_robot_description/urdf/eod_robot_description_left_arm.xacro (robot description, xacro)
@@ -219,6 +219,6 @@
 <link name="Arm_L_end_effector" />
  <joint name="Arm_L_end_effector_joint" type="fixed">
-    <origin xyz="0.001 0.17232 -0.00343" rpy="1.5360 0.4083 3.1307" />
-    <parent link="Arm_L6_link" />
+    <origin xyz="0.0 0.17232 0.0" rpy="1.57079 1.37879 3.14159" />
+    <parent link="Arm_L6_link_add" />
     <child link="Arm_L_end_effector" />
   </joint>

Commit message: urdf_right_arm_rpy

File: eod_robot_description/urdf/eod_robot_description_left_arm.xacro (robot description, xacro)
@@ -180,10 +180,10 @@
     </collision>
   </link>
-  <joint name="Arm_L6_joint" type="continuous">
+  <joint name="Arm_L6_joint" type="revolute">
     <origin xyz="0 0 0.1101" rpy="0 0.4363 0" />
     <parent link="Arm_L5_link" />
     <child link="Arm_L6_link" />
     <axis xyz="0 1 0" />
-    <limit effort="100" velocity="5" />
+    <limit lower="-6.28" upper="6.28" effort="100" velocity="5" />
   </joint>
   <link

File: eod_robot_description/urdf/eod_robot_description_right_arm.xacro (robot description, xacro)
@@ -182,14 +182,15 @@
     </collision>
   </link>
-  <joint name="Arm_R6_joint" type="continuous">
+  <joint name="Arm_R6_joint" type="revolute">
     <origin xyz="0 0 0.1101" rpy="0 -1.74 0" />
     <parent link="Arm_R5_link" />
     <child link="Arm_R6_link" />
     <axis xyz="0 1 0" />
-    <limit effort="100" velocity="5" />
+    <limit lower="-6.28" upper="6.28" effort="100" velocity="5" />
   </joint>
   <link name="Arm_R_end_effector" />
   <joint name="Arm_R_end_effector_joint" type="fixed">
-    <origin xyz="0 0.26797 0" rpy="-1.5708 -1.4008 0" />
+    <!--<origin xyz="0 0.26797 0" rpy="-1.5708 -1.4008 0" />-->
+    <origin xyz="0 0.26797 0" rpy="0 -1.74079 1.5708" />
     <parent link="Arm_R6_link" />
     <child link="Arm_R_end_effector" />
