Commit message: urdf_right_arm_effector_rpy

File: eod_robot_description/urdf/eod_robot_description_right_arm.xacro (robot description, xacro)
@@ -189,11 +189,10 @@
     <limit lower="-6.28" upper="6.28" effort="100" velocity="5" />
   </joint>
-  <link name="Arm_R_end_effector" />
   <joint name="Arm_R_end_effector_joint" type="fixed">
-    <!--<origin xyz="0 0.26797 0" rpy="-1.5708 -1.4008 0" />-->
-    <origin xyz="0 0.26797 0" rpy="0 -1.74079 1.5708" />
+    <origin xyz="0 0.26797 0" rpy="1.5708 1.4008 3.14159" />
     <parent link="Arm_R6_link" />
     <child link="Arm_R_end_effector" />
    </joint>
+  <link name="Arm_R_end_effector" />
   <transmission name="Arm_R1_trans">
     <type>transmission_interface/SimpleTransmission</type>

Commit message: urdf_right_arm_effector_rpy

File: eod_robot_description/urdf/eod_robot_description_right_arm.xacro (robot description, xacro)
@@ -190,5 +190,6 @@
   </joint>
   <joint name="Arm_R_end_effector_joint" type="fixed">
-    <origin xyz="0 0.26797 0" rpy="1.5708 1.4008 3.14159" />
+    <!--<origin xyz="0 0.26797 0" rpy="1.5708 1.4008 3.14159" />-->
+    <origin xyz="0 0.26797 0" rpy="-1.5708 1.74079 0" />
     <parent link="Arm_R6_link" />
     <child link="Arm_R_end_effector" />
